File: plain60-c.sch (KiCad schematic (older format))
At the start: 176 parts, among them J1 HRO-TYPE-C-31-M-12, J2 ISP, K1 KEYSW, K10 KEYSW, K11 KEYSW, K12 KEYSW, K13 KEYSW, K14 KEYSW, K15 KEYSW, K15-1 KEYSW, K16 KEYSW, K17 KEYSW, K18 KEYSW, K19 KEYSW, K2 KEYSW, K20 KEYSW, K21 KEYSW, K22 KEYSW, K23 KEYSW, K24 KEYSW, K25 KEYSW, K26 KEYSW, K27 KEYSW, K28 KEYSW, K29 KEYSW, K3 KEYSW, K31 KEYSW, K31-1 KEYSW, K32 KEYSW, K33 KEYSW, K34 KEYSW, K35 KEYSW, K36 KEYSW, K37 KEYSW, K38 KEYSW, K39 KEYSW, K4 KEYSW, K40 KEYSW, K41 KEYSW, K42 KEYSW, K43 KEYSW, K44 KEYSW, K44-1 KEYSW, K46 KEYSW, K46-1 KEYSW, K47 KEYSW, K48 KEYSW, K49 KEYSW, K5 KEYSW, K50 KEYSW, K51 KEYSW, K52 KEYSW, K53 KEYSW, K54 KEYSW, K55 KEYSW, K56 KEYSW, K57 KEYSW, K58 KEYSW, K58-1 KEYSW, K59 KEYSW, K6 KEYSW, K61 KEYSW, K61-1 KEYSW, K62 KEYSW, K62-1 KEYSW, K63 KEYSW, K63-1 KEYSW, K67 KEYSW, K67-1 KEYSW, K7 KEYSW, K71 KEYSW, K72 KEYSW, K72-1 KEYSW, K73 KEYSW, K73-1 KEYSW, K74 KEYSW, K74-1 KEYSW, K8 KEYSW, K9 KEYSW, SW1 SW_PUSH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

Commit message: Change incorrect ESD chip name and update to more recent Kicad
Parts:
- U2: value USBLC6-2P6 -> USBLC6-2SC6; symbol keyboard_parts:USBLC6-2P6 -> keyboard_parts:USBLC6-2SC6
Changed lines of the file:
@@
 EESchema Schematic File Version 4
-LIBS:plain60-cache
+LIBS:plain60-c-cache
 EELAYER 29 0
 EELAYER END
@@
 $EndComp
 $Comp
-L keyboard_parts:USBLC6-2P6 U2
+L keyboard_parts:USBLC6-2SC6 U2
 U 1 1 5C2DB6C2
 P 3300 1850
 F 0 "U2" H 3300 2175 50  0000 C CNN
-F 1 "USBLC6-2P6" H 3300 2084 50  0000 C CNN
+F 1 "USBLC6-2SC6" H 3300 2084 50  0000 C CNN
 F 2 "Keeb_components:USBLC6-2SC6" H 3000 1550 50  0001 L CNN
 F 3 "" H 3000 1450 50  0001 L CNN

Commit message: Fix bad ISO enter position
Parts:
- K44-1: footprint Keeb_switches:CHERRY_PCB_200H_V_F -> Keeb_switches:CHERRY_PCB_200H_V
Changed lines of the file:
@@
 F 0 "K44-1" H 11950 6950 60  0000 C CNN
 F 1 "KEYSW" H 11950 6850 60  0001 C CNN
-F 2 "Keeb_switches:CHERRY_PCB_200H_V_F" H 11950 6950 60  0001 C CNN
+F 2 "Keeb_switches:CHERRY_PCB_200H_V" H 11950 6950 60  0001 C CNN
 F 3 "" H 11950 6950 60  0000 C CNN
 	1    11950 6950

Commit message: Update to rev2
Parts:
- removed C1, C2: 22p, Keeb_components:C_0805, symbol Device:C
- removed H1: B7, footprints:free_pin, symbol Connector_Generic:Conn_01x01
- added J3: ai03_ud, Keeb_components:JST_SH_SM04B-SRSS-TB_1x04-1MP_P1.00mm_Horizontal, symbol Connector_Generic:Conn_01x04
- added LS1: Speaker, Keeb_components:speaker_AST1109MLTRQ, symbol Device:Speaker
- X1: footprint Keeb_components:crystal_FA238-TSX3225 -> Keeb_components:Resonator_SMD_muRata_CSTNExxV-3Pin-p1.2
- renumbered C3 to C1, C4 to C2, C5 to C3, C6 to C4, C7 to C5, C8 to C6, H2 to H1
Connections:
- net D+: now also J3.2 (Pin_2)
- net D-: now also J3.3 (Pin_3)
- net GND: now also J3.1 (Pin_1), LS1.2
- net VBUS: now also J3.4 (Pin_4)
- net at U1.12 ((OC0A/OC1C/~RTS~/PCINT7)PB7): now also LS1.1
